File: mini-pd-psu/mini-pd-psu.kicad_pcb (KiCad board)
At the start: 4 copper layers, 70 x 60 mm, 34 parts, among them J1 USB_C_Receptacle_USB2.0_16P, J2 Conn_01x02, Q1 AON6264E, Q2 AON6264E, Q3 AON6264E, Q4 AON6264E, U1 ESP32-WROOM-32, U2 STUSB4500QTR, U3 LM5176PWP, U8 TPS62933

Commit message: update
Parts:
- removed J1: USB_C_Receptacle_USB2.0_16P, Connector_USB:USB_C_Receptacle_G-Switch_GT-USB-7010ASV
- added C10: C_Polarized, Capacitor_SMD:CP_Elec_10x10.5, F.Cu at (142.5, 76.6)
- added C11: C_Polarized, Capacitor_SMD:CP_Elec_10x10.5, F.Cu at (153.5, 76.6)
- added C12: 100nF, Capacitor_SMD:C_0603_1608Metric, F.Cu at (155.4, 88.1)
- added C13: 100nF, Capacitor_SMD:C_0603_1608Metric, F.Cu at (156.9, 88.1)
- added C14: 100nF, Capacitor_SMD:C_0603_1608Metric, F.Cu at (159.9, 88.1)
- added C15: C_Polarized, Capacitor_SMD:CP_Elec_10x10.5, F.Cu at (220.3, 124.2)
- added C16: C_Polarized, Capacitor_SMD:CP_Elec_10x10.5, F.Cu at (220.3, 136.2)
- added C17: 10uF, Capacitor_SMD:C_1206_3216Metric, F.Cu at (147.4, 106.3)
- added C19: 10uF, Capacitor_SMD:C_1206_3216Metric, F.Cu at (149.8, 106.3)
- added C21: 10uF, Capacitor_SMD:C_1206_3216Metric, F.Cu at (152.2, 106.3)
- added C22: 10uF, Capacitor_SMD:C_1206_3216Metric, F.Cu at (172.8, 106.3)
- added C23: 1uF, Capacitor_SMD:C_0603_1608Metric, F.Cu at (151.3, 92.2)
- added C24: 100nF, Capacitor_SMD:C_0603_1608Metric, F.Cu at (151.3, 95.2)
- added C26: 100nF, Capacitor_SMD:C_0603_1608Metric, F.Cu at (147.8, 88.1)
- added C29: 1uF, Capacitor_SMD:C_0603_1608Metric, F.Cu at (146.3, 88.1)
- added C30: 100nF, Capacitor_SMD:C_0603_1608Metric, F.Cu at (130.4, 91.5)
- added C31: 10uF, Capacitor_SMD:C_1206_3216Metric, F.Cu at (168.1, 106.3)
- added C32: 10uF, Capacitor_SMD:C_1206_3216Metric, F.Cu at (170.5, 106.3)
- added C33: 100nF, Capacitor_SMD:C_0603_1608Metric, F.Cu at (159.4, 99.9)
- added C5: 100nF, Capacitor_SMD:C_0603_1608Metric, F.Cu at (166.0, 90.4)
- added C7: 1uF, Capacitor_SMD:C_0603_1608Metric, F.Cu at (143.8, 104.7)
- added C8: C_Polarized, Capacitor_SMD:CP_Elec_10x10.5, F.Cu at (220.3, 112.1)
- added C9: C_Polarized, Capacitor_SMD:CP_Elec_10x10.5, F.Cu at (131.5, 76.6)
- added D1: D_Schottky, Diode_SMD:D_0805_2012Metric, F.Cu at (161.5, 101.6)
- added D2: D_Schottky, Diode_SMD:D_0805_2012Metric, F.Cu at (157.2, 101.6)
- added D3: D_Schottky, Diode_SMD:D_0805_2012Metric, F.Cu at (164.6, 84.5)
- added J4: USB_C_Receptacle_USB2.0_16P, Connector_USB:USB_C_Receptacle_GCT_USB4105-xx-A_16P_TopMnt_Horizontal, F.Cu at (113.7, 96.9)
- added R10: 8mR, Resistor_SMD:R_1225_3264Metric, F.Cu at (143.7, 112.5)
- added R13: 100R, Resistor_SMD:R_0603_1608Metric, F.Cu at (144.6, 107.0)
- added R14: 100R, Resistor_SMD:R_0603_1608Metric, F.Cu at (143.0, 107.0)
- added R15: 2K, Resistor_SMD:R_0603_1608Metric, F.Cu at (156.2, 85.8)
- added R16: 100K, Resistor_SMD:R_0603_1608Metric, F.Cu at (153.9, 88.1)
- added R17: 100R, Resistor_SMD:R_0603_1608Metric, F.Cu at (148.7, 92.2)
- added R18: 100R, Resistor_SMD:R_0603_1608Metric, F.Cu at (148.7, 90.7)
- added R19: 93.1K, Resistor_SMD:R_0603_1608Metric, F.Cu at (166.0, 91.9)
- added R20: 93.1K, Resistor_SMD:R_0603_1608Metric, F.Cu at (166.0, 93.4)
- added R5: 8mR, Resistor_SMD:R_1225_3264Metric, F.Cu at (160.3, 106.3)
- added R8: 100R, Resistor_SMD:R_0603_1608Metric, F.Cu at (154.4, 99.8)
- added R9: 100R, Resistor_SMD:R_0603_1608Metric, F.Cu at (152.8, 99.8)
- added U10: OPA376xxDBV, Package_TO_SOT_SMD:SOT-23-5, F.Cu at (150.7, 88.1)
- added U4: DAC8560IxDGK, Package_SON:VSON-8-1EP_3x3mm_P0.65mm_EP1.65x2.4mm, F.Cu at (148.7, 95.2)
- C18: value 22uF -> 47uF; footprint Capacitor_SMD:C_1206_3216Metric -> Capacitor_SMD:CP_Elec_6.3x7.7
- C27: value 22uF -> 10uF
- L2: footprint Inductor_SMD:L_Chilisin_BMRF00101040 -> Inductor_SMD:L_TaiTech_TMPC1265_13.5x12.5mm
- R1: value 115K -> 93.1K
- R2: footprint Resistor_SMD:R_0603_1608Metric -> Resistor_SMD:R_0805_2012Metric
- moved R7 71.6 mm to (129.6, 88.3), turned to -90 degrees
- moved R12 69.7 mm to (131.2, 88.3), turned to 90 degrees
- moved R11 68.2 mm to (132.8, 88.3), turned to -90 degrees
- moved R6 67.2 mm to (134.4, 88.3), turned to -90 degrees
- moved U8 64.9 mm to (133.5, 91.6)
- moved C25 61.5 mm to (136.6, 90.7), turned to 180 degrees
- moved R4 60.9 mm to (136.0, 88.3), turned to 90 degrees
- moved C18 60.7 mm to (130.1, 97.2), turned to -90 degrees
- moved L1 57.7 mm to (136.0, 95.4), turned to -90 degrees
- moved C6 56.4 mm to (136.6, 92.2), turned to 180 degrees
- moved C20 55.3 mm to (136.0, 101.2)
- moved C28 52.9 mm to (136.0, 98.9)
- moved J2 45.9 mm to (123.3, 81.8), turned to 90 degrees
- moved U2 44.2 mm to (122.8, 97.6)
- moved Q2 42.2 mm to (167.4, 112.7)
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Connections:
- C18 pad 1: GND -> VDC
- C18 pad 2: VDC -> GND
- C27 pad 1: GND -> VDC
- C27 pad 2: VDC -> GND
- C3 pad 1: Net-(U3-BOOT2) -> Net-(U3-SW2)
- C3 pad 2: Net-(U3-SW2) -> Net-(D2-K)
- Q2 pad 5: Net-(Q2-D-Pad5) -> VDC
- R1 pad 2: Net-(U3-COMP) -> Net-(U3-MODE)
- R2 pad 2: unconnected-(R2-Pad2) -> Net-(D3-K)
- U3 pad 11: unconnected-(U3-FB-Pad11) -> FB
- U3 pad 12: unconnected-(U3-VOSNS-Pad12) -> BIAS
- U3 pad 13: unconnected-(U3-ISNS(-)-Pad13) -> ISNS-
- U3 pad 14: unconnected-(U3-ISNS(+)-Pad14) -> ISNS+
- U3 pad 15: unconnected-(U3-CSG-Pad15) -> CSG
- U3 pad 16: unconnected-(U3-CS-Pad16) -> CS
- U3 pad 17: unconnected-(U3-PGOOD-Pad17) -> PGOOD
- U3 pad 20: Net-(U3-BOOT2) -> Net-(D2-K)
- U3 pad 23: unconnected-(U3-VCC-Pad23) -> VCC
- U3 pad 24: unconnected-(U3-BIAS-Pad24) -> BIAS
- U3 pad 4: unconnected-(U3-MODE-Pad4) -> Net-(U3-MODE)
- U3 pad 7: unconnected-(U3-SLOPE-Pad7) -> Net-(U3-SLOPE)
Routing:
- net HDRV1: track 0.00 -> 21.5 mm, vias 0 -> 3
- net HDRV2: track 0.00 -> 20.8 mm, vias 0 -> 3
- net LDRV2: track 0.00 -> 14.7 mm, vias 0 -> 3
- net LDRV1: track 0.00 -> 13.3 mm, vias 0 -> 3
- net FB: track 0.00 -> 7.21 mm
- net +3.3V: track 0.00 -> 6.94 mm
- net Net-(U3-VIN): track 0.00 -> 6.01 mm
- net Net-(U8-EN): track 0.00 -> 5.45 mm
- net POWER_EN: track 0.00 -> 4.34 mm
- net Net-(U3-COMP): track 0.00 -> 4.09 mm
- net Net-(D2-K): track 0.00 -> 3.98 mm
- net Net-(D1-K): track 0.00 -> 3.92 mm
- net VDC: track 0.00 -> 3.44 mm
- net Net-(U8-FB): track 0.00 -> 3.39 mm
- net Net-(U10-+): track 0.00 -> 3.34 mm
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- added copper zone on F.Cu, net Net-(C17-Pad1)
- added copper zone on F.Cu, net Net-(Q1-S-Pad1)
- added copper zone on F.Cu, net Net-(U3-SW2)
- added copper zone on F.Cu, net Net-(U8-SW)
- added copper zone on F.Cu, net VDC
- added copper zone on In2.Cu, net VDC

Commit message: update
Parts:
- added R21: 100K, Resistor_SMD:R_0603_1608Metric, F.Cu at (132.1, 106.0)
- added U5: ESP32-S3-MINI-1, RF_Module:ESP32-S2-MINI-1, F.Cu at (161.6, 171.8)
- U1: moved to B.Cu
- moved C1 82.9 mm to (102.3, 110.7)
- moved C16 82.6 mm to (138.6, 124.1), turned to -90 degrees
- moved C15 70.7 mm to (149.6, 124.1), turned to -90 degrees
- moved C8 60.9 mm to (160.6, 124.1), turned to -90 degrees
- moved C20 50.0 mm to (86.6, 93.8)
- moved C28 50.0 mm to (86.6, 91.5)
- moved C30 50.0 mm to (81.0, 84.1)
- moved L1 50.0 mm to (86.6, 88.0)
- moved R11 50.0 mm to (83.4, 80.9)
- moved R4 50.0 mm to (86.6, 80.9)
- moved R6 50.0 mm to (85.0, 80.9)
- moved U8 50.0 mm to (84.1, 84.2)
- moved C18 50.0 mm to (80.7, 89.8)
- moved C25 50.0 mm to (87.2, 83.3)
- moved C6 50.0 mm to (87.2, 84.8)
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Connections:
- U10 pad 1: FB -> Net-(U10--)
- U10 pad 4: FB -> Net-(U10--)
Routing:
- net HDRV1: track 21.5 -> 2.19 mm
- net HDRV2: track 20.8 -> 2.61 mm
- net LDRV2: track 14.7 -> 2.14 mm
- net LDRV1: track 13.3 -> 2.15 mm
- net Net-(U10--): track 0.00 -> 3.36 mm
- net FB: track 7.21 -> 5.35 mm
Other:
- board size 70 x 60 mm -> 70 x 70 mm

Commit message: update
Parts:
- removed U5: ESP32-S3-MINI-1, RF_Module:ESP32-S2-MINI-1
- C10, C11, C15, C16, C8, C9: footprint Capacitor_SMD:CP_Elec_10x10.5 -> Capacitor_SMD:CP_Elec_6.3x5.9
- H1, H2, H3, H4: footprint MountingHole:MountingHole_3.2mm_M3 -> MountingHole:MountingHole_2.2mm_M2
- moved C16 68.2 mm to (201.1, 96.9)
- moved C1 66.2 mm to (168.5, 111.9)
- moved C15 64.6 mm to (208.2, 96.9)
- moved C8 61.1 mm to (215.3, 96.9)
- moved C11 37.9 mm to (189.4, 72.1)
- moved L2 37.2 mm to (138.1, 76.5), turned to 0 degrees
- moved C9 34.7 mm to (175.2, 72.1)
- moved Q2 27.6 mm to (129.1, 87.2), turned to -90 degrees
- moved R10 27.6 mm to (152.8, 87.3), turned to 0 degrees
- moved H3 26.9 mm to (157.5, 117.5)
- moved Q4 23.7 mm to (147.1, 87.2), turned to -90 degrees
- moved Q1 23.2 mm to (135.1, 87.3), turned to 90 degrees
- moved R14 22.8 mm to (153.6, 92.8), turned to 90 degrees
- moved Q3 21.7 mm to (141.1, 87.3), turned to 90 degrees
- moved D3 21.3 mm to (131.3, 114.9), turned to -90 degrees
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Connections:
- J4 pad S1: GND -> unconnected-(J4-SHIELD-PadS1)_3
Routing:
- removed copper zone on B.Cu, net GND
- removed copper zone on F.Cu, net GND
- removed copper zone on In1.Cu, net GND
- removed copper zone on In2.Cu, net VDC
Other:
- board size 70 x 70 mm -> 50 x 50 mm
