File: mini-pd-psu/mini-pd-psu.kicad_sch (KiCad schematic)
At the start: 37 parts, among them J1 USB_C_Receptacle_USB2.0_16P, J2 Conn_01x02, J3 Conn_01x08, Q1 AON6264E, Q2 AON6264E, Q3 AON6264E, Q4 AON6264E, Q5 AON6264E, Q6 AON6264E, U1 ESP32-WROOM-32, U2 STUSB4500QTR, U3 LM5176PWP, U8 TPS62933

Commit message: update
Parts:
- removed C18: 22uF, Capacitor_SMD:C_1206_3216Metric, symbol Device:C
- removed J1: USB_C_Receptacle_USB2.0_16P, Connector_USB:USB_C_Receptacle_G-Switch_GT-USB-7010ASV, symbol Connector:USB_C_Receptacle_USB2.0_16P
- removed Q5, Q6: AON6264E, Package_DFN_QFN:PQFN-8-EP_6x5mm_P1.27mm_Generic, symbol TiManh:NMOS-8PINS
- added C10, C11, C15, C16, C8, C9: C_Polarized, Capacitor_SMD:CP_Elec_10x10.5, symbol Device:C_Polarized
- added C12, C13, C14, C24, C26, C30, C5: 100nF, Capacitor_SMD:C_0603_1608Metric, symbol Device:C
- added C17, C19, C21, C22, C31, C32: 10uF, Capacitor_SMD:C_1206_3216Metric, symbol Device:C
- added C18: 47uF, Capacitor_SMD:CP_Elec_6.3x7.7, symbol Device:C_Polarized
- added C23, C29, C7: 1uF, Capacitor_SMD:C_0603_1608Metric, symbol Device:C
- added C33: 100nF, Capacitor_SMD:C_0603_1608Metric, symbol Device:C_Small
- added D1, D2, D3: D_Schottky, Diode_SMD:D_0805_2012Metric, symbol Device:D_Schottky
- added J4: USB_C_Receptacle_USB2.0_16P, Connector_USB:USB_C_Receptacle_GCT_USB4105-xx-A_16P_TopMnt_Horizontal, symbol Connector:USB_C_Receptacle_USB2.0_16P
- added R10, R5: 8mR, Resistor_SMD:R_1225_3264Metric, symbol Device:R
- added R13, R14, R17, R18, R8, R9: 100R, Resistor_SMD:R_0603_1608Metric, symbol Device:R_Small
- added R15: 2K, Resistor_SMD:R_0603_1608Metric, symbol Device:R_Small
- added R16: 100K, Resistor_SMD:R_0603_1608Metric, symbol Device:R_Small
- added R19, R20: 93.1K, Resistor_SMD:R_0603_1608Metric, symbol Device:R_Small
- added U10: OPA376xxDBV, Package_TO_SOT_SMD:SOT-23-5, symbol Amplifier_Operational:OPA376xxDBV
- added U4: DAC8560IxDGK, Package_SON:VSON-8-1EP_3x3mm_P0.65mm_EP1.65x2.4mm, symbol Analog_DAC:DAC8560IxDGK
- C27: value 22uF -> 10uF
- L2: footprint Inductor_SMD:L_Chilisin_BMRF00101040 -> Inductor_SMD:L_TaiTech_TMPC1265_13.5x12.5mm
- R1: value 115K -> 93.1K
- R2: footprint Resistor_SMD:R_0603_1608Metric -> Resistor_SMD:R_0805_2012Metric
Connections:
- net +3.3V: now also C23.2, C24.2, C26.2, C29.2, U10.2 (V-), U4.1 (V_{DD})
- net GND: now also C27.2, C10.2, C11.2, C13.1, C14.1, C15.2, C16.2, C17.2, C18.2, C19.2, C21.2, C22.2, C23.1, C24.1, C26.1, C29.1, C30.1, C31.2, C32.2, C33.1, C5.1, C8.2, C9.2, J4.A1 (GND), J4.A12 (GND), J4.B1 (GND), J4.B12 (GND), J4.S1 (SHIELD), R15.1, R18.2, R20.1, R5.2, R9.1, U10.5 (V+), U4.8 (GND); no longer C27.1
- net POWER_EN: now also R19.1, R20.2
- net VDC: now also C27.1, Q2.5 (D), Q2.6 (D), Q2.7 (D), Q2.8 (D), C10.1, C11.1, C18.1, C22.1, C30.2, C31.1, C32.1, C9.1, D3.2 (A), J4.A4 (VBUS), J4.A9 (VBUS), J4.B4 (VBUS), J4.B9 (VBUS), R19.2; no longer C27.2
- net at R1.2: now also U3.4 (MODE); no longer U3.9 (COMP)
- net at C2.1, U3.26 (BOOT1): now also D1.1 (K)
- net at L2.2, Q3.5 (D), Q3.6 (D)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: now also C3.1; no longer C3.2
- net at Q4.5 (D), Q4.6 (D), Q4.7 (D)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: now also C17.1, C19.1, C21.1, R10.1, R13.2
- net FB: now reaches U3.11 (FB)
- net FB: now also R16.2, U10.1, U10.4 (-)
- net BIAS: now reaches U3.12 (VOSNS)
- net BIAS: now also U3.24 (BIAS), C15.1, C16.1, C33.2, C8.1, R10.2, R14.2, R16.1
- net ISNS-: now reaches U3.13 (ISNS(-))
- net ISNS-: now also C7.1, R14.1
- net ISNS+: now reaches U3.14 (ISNS(+))
- net ISNS+: now also C7.2, R13.1
- net CSG: now reaches U3.15 (CSG)
- net CSG: now also R9.2
- net CS: now reaches U3.16 (CS)
- net CS: now also R8.2
- net PGOOD: now reaches U3.17 (PGOOD)
- net at R2.1, U3.2 (VIN): now also C5.2
- net at U3.20 (BOOT2): now also C3.2, D2.1 (K); no longer C3.1
- net VCC: now reaches U3.23 (VCC)
- net VCC: now also D1.2 (A), D2.2 (A)
- net at U3.7 (SLOPE): now also C14.2
- net at Q1.1 (S), Q1.2 (S), Q1.3 (S)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: now also R5.1, R8.1
- net at R2.2: now also D3.1 (K)
- new net: J4.A6 (D+), J4.B6 (D+)
- new net: J4.A7 (D-), J4.B7 (D-)
- new net: C12.2, C13.2, U3.9 (COMP)
- new net: C12.1, R15.2
- new net: R17.2, R18.1, U10.3 (+)
- new net: R17.1, U4.3 (V_{FB}), U4.4 (V_{OUT})
- no-connect marks 0 -> 1
Other:
- moved on the sheet: C1, C2, C20, C25, C28, C3, C4, C6, H1, H2, H3, H4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

Commit message: update
Parts:
- added R21: 100K, Resistor_SMD:R_0603_1608Metric, symbol Device:R_Small
- added U5: ESP32-S3-MINI-1, RF_Module:ESP32-S2-MINI-1, symbol RF_Module:ESP32-S3-MINI-1
Connections:
- net FB: now also R21.1; no longer U10.1, U10.4 (-)
- net GND: now also U5.1 (GND), U5.2 (GND), U5.42 (GND), U5.43 (GND), U5.46 (GND), U5.47 (GND), U5.48 (GND), U5.49 (GND), U5.50 (GND), U5.51 (GND), U5.52 (GND), U5.53 (GND), U5.54 (GND), U5.55 (GND), U5.56 (GND), U5.57 (GND), U5.58 (GND), U5.59 (GND), U5.60 (GND), U5.61 (GND), U5.62 (GND), U5.63 (GND), U5.64 (GND), U5.65 (GND); no longer J4.S1 (SHIELD)
- new net: R21.2, U10.1, U10.4 (-)
- no-connect marks 1 -> 2

Commit message: update
Parts:
- removed U5: ESP32-S3-MINI-1, RF_Module:ESP32-S2-MINI-1, symbol RF_Module:ESP32-S3-MINI-1
- C10, C11, C15, C16, C8, C9: footprint Capacitor_SMD:CP_Elec_10x10.5 -> Capacitor_SMD:CP_Elec_6.3x5.9
- H1, H2, H3, H4: footprint MountingHole:MountingHole_3.2mm_M3 -> MountingHole:MountingHole_2.2mm_M2
Other:
- moved on the sheet: C1, J4, U2
