File: PCB/mini-pd-psu.kicad_pcb (KiCad board)
At the start: 2 copper layers, 50 x 50 mm, 55 parts, among them J1 Conn_01x02, J2 Conn_01x02, J4 USB_C_Receptacle_USB2.0_16P, J5 Conn_01x02, Q1 NMOS-8PINS, Q2 NMOS-8PINS, U1 STM32G431RBTx, U2 STUSB4500QTR, U3 LM3150MH, U8 TPS62933

Commit message: update
Parts:
- added C31: 47uF, Capacitor_SMD:CP_Elec_6.3x5.9, F.Cu at (115.0, 95.0)
- added C32: 47uF, Capacitor_SMD:CP_Elec_6.3x5.9, F.Cu at (153.2, 78.0)
- added C33: 100nF, Capacitor_SMD:C_0603_1608Metric, F.Cu at (145.2, 104.9)
- added C34: 100nF, Capacitor_SMD:C_0603_1608Metric, F.Cu at (146.7, 104.9)
- added R10: 1K, Resistor_SMD:R_0603_1608Metric, F.Cu at (145.2, 107.9)
- added R8: 1K, Resistor_SMD:R_0603_1608Metric, F.Cu at (142.2, 107.9)
- added R9: 1K, Resistor_SMD:R_0603_1608Metric, F.Cu at (143.7, 107.9)
- added U4: STM32G431CBUx, Package_DFN_QFN:QFN-48-1EP_7x7mm_P0.5mm_EP5.6x5.6mm, F.Cu at (136.2, 104.0)
- C10, C19: value C_Polarized -> 47uF
- U1: value STM32G431RBTx -> STM32G431KBUx; footprint Package_QFP:LQFP-64_10x10mm_P0.5mm -> Package_DFN_QFN:QFN-32-1EP_5x5mm_P0.5mm_EP3.45x3.45mm
- U2: value STUSB4500QTR -> FUSB302BMPX; footprint Package_DFN_QFN:QFN-24-1EP_4x4mm_P0.5mm_EP2.7x2.7mm -> Package_DFN_QFN:WQFN-14-1EP_2.5x2.5mm_P0.5mm_EP1.45x1.45mm
- moved C1 38.5 mm to (130.2, 101.3), turned to 180 degrees
- moved C11 36.9 mm to (138.6, 87.9)
- moved U1 36.4 mm to (114.7, 133.0)
- moved C23 36.0 mm to (130.2, 99.7), turned to 180 degrees
- moved J1 31.4 mm to (146.6, 92.5)
- moved C22 29.5 mm to (148.6, 112.9), turned to 0 degrees
- moved C26 29.2 mm to (139.0, 109.7), turned to -90 degrees
- moved R7 29.1 mm to (152.5, 117.2), turned to 0 degrees
- moved R12 28.3 mm to (152.5, 118.8), turned to 0 degrees
- moved C21 26.9 mm to (148.6, 115.2), turned to 0 degrees
- moved C30 26.6 mm to (149.4, 117.2), turned to 180 degrees
- moved C5 26.4 mm to (124.5, 73.5)
- moved C13 26.2 mm to (127.0, 73.5)
- moved U2 25.5 mm to (148.0, 108.2), turned to -90 degrees
- moved J4 25.3 mm to (156.3, 108.5)
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Connections:
- C19 pad 1: VBUS -> VDC
- C21 pad 2: VBUS -> VDC
- C22 pad 2: VBUS -> VDC
- J4 pad A5: unconnected-(J4-CC1-PadA5) -> Net-(J4-CC1)
- J4 pad B5: unconnected-(J4-CC2-PadB5) -> Net-(J4-CC2)
- J4 pad S1: unconnected-(J4-SHIELD-PadS1)_3 -> GND
- J5 pad 2: VBUS -> +5V
- U1 pad 1: +3.3V -> Net-(U1-VDDA)
- U1 pad 14: unconnected-(U1-PA2-Pad14) -> GND
- U1 pad 15: GND -> Net-(U1-VDDA)
- U1 pad 16: +3.3V -> GND
- U1 pad 17: unconnected-(U1-PA3-Pad17) -> Net-(U1-VDDA)
- U1 pad 27: GND -> unconnected-(U1-PB4-Pad27)
- U1 pad 28: +3.3V -> unconnected-(U1-PB5-Pad28)
- U1 pad 29: +3.3V -> unconnected-(U1-PB6-Pad29)
- U1 pad 31: GND -> unconnected-(U1-PB8-Pad31)
- U1 pad 32: +3.3V -> GND
- U1 pad 33: unconnected-(U1-PB11-Pad33) -> GND
- U2 pad 1: unconnected-(U2-CC1DB-Pad1) -> Net-(J4-CC2)
- U2 pad 10: GND -> Net-(J4-CC1)
- U2 pad 11: unconnected-(U2-ATTACH-Pad11) -> Net-(J4-CC1)
- U2 pad 14: unconnected-(U2-POWER_OK3-Pad14) -> Net-(J4-CC2)
- U2 pad 15: unconnected-(U2-GPIO-Pad15) -> GND
- U2 pad 2: unconnected-(U2-CC1-Pad2) -> VDC
- U2 pad 3: unconnected-(U2-NC-Pad3) -> +3.3V
- U2 pad 4: unconnected-(U2-CC2-Pad4) -> +3.3V
- U2 pad 5: unconnected-(U2-CC2DB-Pad5) -> Net-(U2-INT_N)
- U2 pad 6: unconnected-(U2-RESET-Pad6) -> Net-(U2-SCL)
- U2 pad 7: unconnected-(U2-SCL-Pad7) -> Net-(U2-SDA)
- U2 pad 8: unconnected-(U2-SDA-Pad8) -> GND
- U2 pad 9: unconnected-(U2-DISCH-Pad9) -> GND
Routing:
- net VBUS: track 30.3 -> 1.55 mm
- net VDC: track 5.95 -> 13.8 mm, vias 0 -> 8
- net Net-(J4-CC1): track 0.00 -> 4.81 mm
- net Net-(J4-CC2): track 0.00 -> 4.81 mm
- net Net-(Q2-G): track 9.06 -> 4.73 mm
- net Net-(Q2-D): track 8.04 -> 11.9 mm
- net Net-(Q1-G): track 5.23 -> 8.30 mm
- net Net-(U8-EN): track 3.10 -> 5.93 mm
- net Net-(J4-D--PadA7): track 0.00 -> 2.44 mm
- net Net-(J4-D+-PadA6): track 0.00 -> 2.44 mm
- net +3.3V: track 0.00 -> 2.38 mm
- net Net-(U3-SS): track 2.17 -> 4.03 mm
- net Net-(U3-ILIM): track 3.83 -> 2.02 mm
- net Net-(U3-VCC): track 0.00 -> 1.68 mm
- net Net-(U3-FB): track 3.82 -> 5.35 mm
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- added copper zone on B.Cu, net VDC
Other:
- board text added: "HI"

Commit message: update
Parts:
- added C35: 47uF, Capacitor_SMD:CP_Elec_6.3x5.9, F.Cu at (124.7, 131.2)
- added R13: R, Resistor_SMD:R_2512_6332Metric, F.Cu at (135.5, 94.1)
- added R14: R, Resistor_SMD:R_2512_6332Metric, F.Cu at (146.3, 84.4)
- added R15: R, Resistor_SMD:R_2512_6332Metric, F.Cu at (128.5, 107.1)
- added SW1: RotaryEncoder, TiManh:EC05E1220401, F.Cu at (136.0, 117.1)
- added SW4: SW_Push_45deg, Button_Switch_THT:SW_Tactile_SKHH_Angled, F.Cu at (175.2, 129.6)
- added SW9: SW_Push_45deg, Button_Switch_THT:SW_Tactile_SKHH_Angled, F.Cu at (188.2, 137.8)
- added U5: INA3221, Package_DFN_QFN:Texas_RGV0016A_VQFN-16-1EP_4x4mm_P0.65mm_EP2.1x2.1mm, F.Cu at (141.2, 94.1)
- moved U1 67.6 mm to (175.3, 103.0)
- moved U4 39.2 mm to (97.7, 111.4)
- moved C24 39.2 mm to (103.5, 108.8)
- moved C1 39.2 mm to (91.7, 108.7)
- moved C23 39.2 mm to (91.7, 107.1)
- moved C26 34.6 mm to (105.2, 117.1)
- moved R10 30.4 mm to (175.2, 112.8)
- moved R8 30.4 mm to (172.2, 112.8)
- moved R9 30.4 mm to (173.7, 112.8)
- moved C33 28.6 mm to (173.5, 109.3)
- moved C34 28.6 mm to (175.0, 109.3)
- moved C14 24.1 mm to (121.6, 73.5)
- moved C20 19.8 mm to (146.4, 132.9)
- moved C22 19.8 mm to (154.4, 131.8)
- moved C28 19.8 mm to (144.1, 132.9)
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Connections:
- C10 pad 1: VBUS -> SENSE_OUT+
- C11 pad 1: VBUS -> SENSE_OUT+
- C14 pad 2: VBUS -> SENSE_OUT+
- C15 pad 2: VBUS -> SENSE_OUT+
- C16 pad 2: VBUS -> SENSE_OUT+
- C17 pad 2: VBUS -> SENSE_OUT+
- C18 pad 2: VBUS -> SENSE_OUT+
- C31 pad 1: VBUS -> SENSE_OUT+
- J1 pad 2: VDC -> Net-(J1-Pin_2)
- J2 pad 2: VBUS -> SENSE_OUT+
- J4 pad A4: VDC -> Net-(J1-Pin_2)
- J4 pad A9: VDC -> Net-(J1-Pin_2)
- J4 pad B4: VDC -> Net-(J1-Pin_2)
- J4 pad B9: VDC -> Net-(J1-Pin_2)
- J5 pad 2: +5V -> Net-(J5-Pin_2)
- L2 pad 2: VBUS -> SENSE_OUT-
- R3 pad 2: VBUS -> SENSE_OUT+
- U2 pad 2: VDC -> Net-(J1-Pin_2)
Routing:
- net SENSE_OUT+: track 0.00 -> 9.58 mm
- net SENSE_OUT-: track 0.00 -> 4.69 mm, vias 0 -> 2
- net VBUS: track 1.55 -> 0.00 mm
- net VDC: track 13.8 -> 13.0 mm, vias 8 -> 0
- net GND: vias 81 -> 52
- added copper zone on B.Cu, net Net-(J1-Pin_2)
- added copper zone on F.Cu, net Net-(J1-Pin_2)
- added copper zone on F.Cu, net SENSE_OUT+
- added copper zone on F.Cu, net SENSE_OUT-
- removed copper zone on F.Cu, net VBUS
- removed copper zone on B.Cu, net VDC
Other:
- outline, holes or cut-outs redrawn

Commit message: update
Parts:
- removed SW1: RotaryEncoder, TiManh:EC05E1220401
- removed SW4, SW9: SW_Push_45deg, Button_Switch_THT:SW_Tactile_SKHH_Angled
- added C36: 100nF, Capacitor_SMD:C_0603_1608Metric, F.Cu at (149.1, 84.4)
- added U6: MT6701CT, Package_SO:SOIC-8_3.9x4.9mm_P1.27mm, F.Cu at (135.0, 115.0)
- H1, H2, H3, H4: value MountingHole -> MountingHole_Pad; footprint MountingHole:MountingHole_2.2mm_M2 -> MountingHole:MountingHole_2.2mm_M2_Pad_Via
- J2, J5: footprint Connector_AMASS:AMASS_XT30PW-M_1x02_P2.50mm_Horizontal -> Connector_AMASS:AMASS_XT30PW-F_1x02_P2.50mm_Horizontal
- moved C24 96.8 mm to (192.7, 146.6)
- moved C26 96.8 mm to (194.4, 154.9)
- moved U4 96.8 mm to (186.9, 149.2)
- moved C1 96.8 mm to (180.9, 146.4)
- moved C23 96.8 mm to (180.9, 144.8)
- moved C33 26.7 mm to (147.2, 104.5)
- moved C34 26.6 mm to (148.8, 104.5)
- moved C16 23.7 mm to (117.9, 78.5), turned to -90 degrees
- moved C10 22.4 mm to (113.0, 74.0), turned to 180 degrees
- moved C18 21.2 mm to (120.2, 78.5), turned to -90 degrees
- moved C4 20.3 mm to (119.3, 73.5)
- moved C17 19.6 mm to (122.5, 78.5), turned to -90 degrees
- moved C15 18.9 mm to (124.8, 78.5), turned to -90 degrees
- moved C27 17.1 mm to (178.4, 117.6)
- moved C29 17.1 mm to (178.4, 120.2)
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Connections:
- C10 pad 1: SENSE_OUT+ -> SENSE2-
- C11 pad 1: SENSE_OUT+ -> SENSE2-
- C13 pad 2: VDC -> SENSE1-
- C14 pad 2: SENSE_OUT+ -> SENSE2-
- C15 pad 2: SENSE_OUT+ -> SENSE2-
- C16 pad 2: SENSE_OUT+ -> SENSE2-
- C17 pad 2: SENSE_OUT+ -> SENSE2-
- C18 pad 2: SENSE_OUT+ -> SENSE2-
- C19 pad 1: VDC -> SENSE1-
- C2 pad 2: VDC -> SENSE1-
- C21 pad 2: VDC -> SENSE1-
- C22 pad 2: VDC -> SENSE1-
- C3 pad 2: VDC -> SENSE1-
- C30 pad 2: VDC -> SENSE1-
- C31 pad 1: SENSE_OUT+ -> SENSE2-
- C32 pad 1: VDC -> SENSE1-
- C4 pad 2: VDC -> SENSE1-
- C5 pad 2: VDC -> SENSE1-
- C8 pad 1: VDC -> SENSE1-
- J1 pad 2: Net-(J1-Pin_2) -> SENSE1+
- J2 pad 2: SENSE_OUT+ -> SENSE2-
- J4 pad A4: Net-(J1-Pin_2) -> SENSE1+
- J4 pad A9: Net-(J1-Pin_2) -> SENSE1+
- J4 pad B4: Net-(J1-Pin_2) -> SENSE1+
- J4 pad B9: Net-(J1-Pin_2) -> SENSE1+
- L2 pad 2: SENSE_OUT- -> SENSE2+
- Q1 pad 5: VDC -> SENSE1-
- R13 pad 1: SENSE_OUT- -> SENSE2+
- R13 pad 2: SENSE_OUT+ -> SENSE2-
- R14 pad 1: Net-(J1-Pin_2) -> SENSE1+
- R14 pad 2: VDC -> SENSE1-
- R2 pad 2: VDC -> SENSE1-
- R3 pad 2: SENSE_OUT+ -> SENSE2-
- R7 pad 2: VDC -> SENSE1-
- U2 pad 2: Net-(J1-Pin_2) -> SENSE1+
- U3 pad 2: VDC -> SENSE1-
- U5 pad 1: unconnected-(U5-IN-3-Pad1) -> SENSE3-
- U5 pad 11: SENSE_OUT- -> SENSE1-
- U5 pad 12: SENSE_OUT+ -> SENSE1+
- U5 pad 14: unconnected-(U5-IN-2-Pad14) -> SENSE2-
- U5 pad 15: unconnected-(U5-IN+2-Pad15) -> SENSE2+
- U5 pad 2: unconnected-(U5-IN+3-Pad2) -> SENSE3+
- U8 pad 3: VDC -> SENSE1-
Routing:
- net VDC: track 13.0 -> 0.00 mm
- net SENSE1-: track 0.00 -> 9.81 mm, vias 0 -> 2
- net SENSE_OUT+: track 9.58 -> 0.00 mm
- net Net-(U8-FB): track 8.13 -> 0.00 mm
- net Net-(U8-EN): track 5.93 -> 0.00 mm
- net SENSE_OUT-: track 4.69 -> 0.00 mm, vias 2 -> 0
- net SENSE2-: track 0.00 -> 1.55 mm
- net GND: vias 52 -> 14
- added copper zone on B.Cu, net SENSE1+
- added copper zone on F.Cu, net SENSE1+
- added copper zone on F.Cu, net SENSE1-
- added copper zone on F.Cu, net SENSE2+
- added copper zone on F.Cu, net SENSE2-
- removed copper zone on B.Cu, net Net-(J1-Pin_2)
- removed copper zone on F.Cu, net Net-(J1-Pin_2)
- removed copper zone on F.Cu, net SENSE_OUT+
- removed copper zone on F.Cu, net SENSE_OUT-
- removed copper zone on F.Cu, net VDC
Other:
- board size 50 x 50 mm -> 60 x 50 mm
