File: PCB/mini-pd-psu.kicad_sch (KiCad schematic)
At the start: 56 parts, among them J1 Conn_01x02, J2 Conn_01x02, J3 Conn_01x08, J4 USB_C_Receptacle_USB2.0_16P, J5 Conn_01x02, Q1 NMOS-8PINS, Q2 NMOS-8PINS, U1 STM32G431RBTx, U2 STUSB4500QTR, U3 LM3150MH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

Commit message: update
Parts:
- removed U1: STM32G431RBTx, Package_QFP:LQFP-64_10x10mm_P0.5mm, symbol MCU_ST_STM32G4:STM32G431RBTx
- removed U2: STUSB4500QTR, Package_DFN_QFN:QFN-24-1EP_4x4mm_P0.5mm_EP2.7x2.7mm, symbol Interface_USB:STUSB4500QTR
- added C31, C32: 47uF, Capacitor_SMD:CP_Elec_6.3x5.9, symbol Device:C_Polarized
- added C33, C34: 100nF, Capacitor_SMD:C_0603_1608Metric, symbol Device:C
- added R10, R8, R9: 1K, Resistor_SMD:R_0603_1608Metric, symbol Device:R_Small
- added U1: STM32G431KBUx, Package_DFN_QFN:QFN-32-1EP_5x5mm_P0.5mm_EP3.45x3.45mm, symbol MCU_ST_STM32G4:STM32G431KBUx
- added U2: FUSB302BMPX, Package_DFN_QFN:WQFN-14-1EP_2.5x2.5mm_P0.5mm_EP1.45x1.45mm, symbol Interface_USB:FUSB302BMPX
- added U4: STM32G431CBUx, Package_DFN_QFN:QFN-48-1EP_7x7mm_P0.5mm_EP5.6x5.6mm, symbol MCU_ST_STM32G4:STM32G431CBUx
- C10, C19: value C_Polarized -> 47uF
Connections:
- net +3.3V: now also C33.1, C34.1, R10.2, R8.2, R9.2, U2.3 (VDD), U2.4 (VDD), U4.1 (VBAT), U4.21 (VDDA), U4.23 (VDD), U4.35 (VDD), U4.48 (VDD)
- net +5V: now also J5.2 (Pin_2)
- net GND: now also J4.S1 (SHIELD), C31.2, C32.2, C33.2, C34.2, U1.14 (VSSA), U1.16 (VSS), U1.32 (VSS), U1.33 (VSS), U2.15 (GND), U2.8 (GND), U2.9 (GND)
- net VBUS: now also C31.1; no longer C19.1, C21.2, C22.2, J5.2 (Pin_2)
- net VDC: now also C19.1, C21.2, C22.2, C32.1, U2.2 (VBUS)
- net at J4.A5 (CC1): now also U2.10 (CC1), U2.11 (CC1)
- net at J4.B5 (CC2): now also U2.1 (CC2), U2.14 (CC2)
- new net: U1.1 (VDD), U1.15 (VDDA), U1.17 (VDD)
- new net: R9.1, U2.6 (SCL)
- new net: R8.1, U2.7 (SDA)
- new net: R10.1, U2.5 (INT_N)
- no-connect marks 1 -> 0

Commit message: update
Parts:
- added C35: 47uF, Capacitor_SMD:CP_Elec_6.3x5.9, symbol Device:C_Polarized
- added R13, R14, R15: R, Resistor_SMD:R_2512_6332Metric, symbol Device:R
- added SW1: RotaryEncoder, TiManh:EC05E1220401, symbol Device:RotaryEncoder
- added SW2, SW3: SW_Push, symbol Switch:SW_Push
- added U5: INA3221, Package_DFN_QFN:Texas_RGV0016A_VQFN-16-1EP_4x4mm_P0.65mm_EP2.1x2.1mm, symbol Power_Management:INA3221
Connections:
- net +5V: now also R15.2; no longer J5.2 (Pin_2)
- net GND: now also C35.2, U5.17 (EP), U5.3 (GND)
- net VBUS: now also R13.2, U5.12 (IN+1); no longer L2.2
- net VDC: now also R14.2; no longer J1.2 (Pin_2), J4.A4 (VBUS), J4.A9 (VBUS), J4.B4 (VBUS), J4.B9 (VBUS), U2.2 (VBUS)
- new net: J1.2 (Pin_2), J4.A4 (VBUS), J4.A9 (VBUS), J4.B4 (VBUS), J4.B9 (VBUS), R14.1, U2.2 (VBUS)
- new net: C35.1, J5.2 (Pin_2), R15.1
- new net SENSE_OUT-: L2.2, R13.1, U5.11 (IN-1)
Other:
- moved on the sheet: J1, L2

Commit message: update
Parts:
- removed H1, H2, H3, H4: MountingHole, MountingHole:MountingHole_2.2mm_M2, symbol Mechanical:MountingHole
- removed SW1: RotaryEncoder, TiManh:EC05E1220401, symbol Device:RotaryEncoder
- added C36: 100nF, Capacitor_SMD:C_0603_1608Metric, symbol Device:C
- added H1, H2, H3, H4: MountingHole_Pad, MountingHole:MountingHole_2.2mm_M2_Pad_Via, symbol Mechanical:MountingHole_Pad
- added U6: MT6701CT, Package_SO:SOIC-8_3.9x4.9mm_P1.27mm, symbol Sensor_Magnetic:MT6701CT
- J2, J5: footprint Connector_AMASS:AMASS_XT30PW-M_1x02_P2.50mm_Horizontal -> Connector_AMASS:AMASS_XT30PW-F_1x02_P2.50mm_Horizontal
Connections:
- net VBUS: now also U5.14 (IN-2); no longer U5.12 (IN+1)
- net VDC: now also U5.11 (IN-1), C36.2
- net SENSE3-: now reaches U5.1 (IN-3)
- net SENSE2+: now reaches U5.15 (IN+2)
- net SENSE2+: now also L2.2, R13.1
- net SENSE3+: now reaches U5.2 (IN+3)
- net SENSE1+: now reaches J1.2 (Pin_2), J4.A4 (VBUS), J4.A9 (VBUS), J4.B4 (VBUS), J4.B9 (VBUS), R14.1, U2.2 (VBUS)
- net SENSE1+: now also U5.12 (IN+1), C36.1
- removed net SENSE_OUT-: L2.2, R13.1, U5.11 (IN-1)
Other:
- moved on the sheet: C1, C10, C11, C12, C13, C14, C15, C16, C17, C18, C19, C2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
